File: Gamma-Boards/Gamma-32ch-3in/Gamma-32ch-3in.kicad_pcb (KiCad board)
At the start: 2 copper layers, 116.5 x 80.1 mm, 99 parts

Commit message: Fixed Gamma-32ch-3in
Parts:
- removed the ? at (183.6, 103.9)
Connections:
- REF** pad 1: (no net) -> 24C
- REF** pad 2: (no net) -> 24A
- REF** pad 15: (no net) -> 23C
Routing:
- net 23C: track 16.4 -> 103.9 mm, vias 1 -> 2
- net 24A: track 107.0 -> 106.0 mm
