File: IV_Boards/IV_Board_9ch_latch/IV_Board_9ch_latch.kicad_pcb (KiCad board)
At the start: 2 copper layers, 99.2 x 25.2 mm, 10 parts

Commit message: Edge Card 9ch v2 + 9ch latch IV board v2 +
Updated Edge Card 9ch to v2 with expanded pads, and fixed 9ch latch IV board to reroute one trace around a hole
Connections:
- REF** pad 11: A37 -> A5
Routing:
- net A5: track 45.3 -> 46.4 mm
Other:
- board text added: "IV Board 9ch latch v2"
- board text removed: "IV Board 9ch latch"
Changed lines of the file:
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@@
 	(net 27 "A36")
 	(net 28 "K36")
-	(net 29 "A37")
-	(net 30 "K37")
-	(net 31 "A38")
-	(net 32 "K38")
-	(net 33 "A39")
-	(net 34 "K39")
-	(net 35 "GND")
+	(net 29 "K37")
+	(net 30 "A38")
+	(net 31 "K38")
+	(net 32 "A39")
+	(net 33 "K39")
+	(net 34 "GND")
 	(footprint "Connector_Coaxial:SMA_Amphenol_901-144_Vertical"
 		(layer "F.Cu")
@@
 			(layers "F.Cu" "F.Mask" "F.Paste")
 			(roundrect_rratio 0.25)
-			(net 29 "A37")
+			(net 15 "A5")
 		)
 		(pad "12" smd roundrect
@@
 			(layers "F.Cu" "F.Mask" "F.Paste")
 			(roundrect_rratio 0.25)
-			(net 30 "K37")
+			(net 29 "K37")
 		)
 		(pad "13" smd roundrect
@@
 			(layers "F.Cu" "F.Mask" "F.Paste")
 			(roundrect_rratio 0.25)
-			(net 31 "A38")
+			(net 30 "A38")
 		)
 		(pad "14" smd roundrect
@@
 			(layers "F.Cu" "F.Mask" "F.Paste")
 			(roundrect_rratio 0.25)
-			(net 32 "K38")
+			(net 31 "K38")
 		)
 		(pad "15" smd roundrect
@@
 			(layers "F.Cu" "F.Mask" "F.Paste")
 			(roundrect_rratio 0.25)
-			(net 33 "A39")
+			(net 32 "A39")
 		)
 		(pad "16" smd roundrect
@@
 			(layers "F.Cu" "F.Mask" "F.Paste")
 			(roundrect_rratio 0.25)
-			(net 34 "K39")
+			(net 33 "K39")
 		)
 		(pad "17" smd roundrect
@@
 			(layers "F.Cu" "F.Mask" "F.Paste")
 			(roundrect_rratio 0.25)
-			(net 35 "GND")
+			(net 34 "GND")
 		)
 		(pad "18" smd roundrect
@@
 			(layers "F.Cu" "F.Mask" "F.Paste")
 			(roundrect_rratio 0.25)
-			(net 35 "GND")
+			(net 34 "GND")
 		)
 		(embedded_fonts no)
@@
 		)
 	)
-	(gr_text "IV Board 9ch latch"
+	(gr_text "IV Board 9ch latch v2"
 		(at 207.2 112.2 0)
 		(layer "F.SilkS")
@@
 	)
 	(segment
-		(start 205.525 95.675)
-		(end 207.875 95.675)
+		(start 206.749248 95.674)
+		(end 208.075248 97)
 		(width 0.2)
 		(layer "F.Cu")
@@
 	)
 	(segment
-		(start 188 96.2)
-		(end 192.434314 96.2)
+		(start 208.075248 97)
+		(end 218.2 97)
 		(width 0.2)
 		(layer "F.Cu")
@@
 	)
 	(segment
-		(start 176.749 96.099)
-		(end 179.758451 96.099)
+		(start 193.3589 95.274)
+		(end 195.1661 95.274)
 		(width 0.2)
 		(layer "F.Cu")
@@
 	)
 	(segment
-		(start 186.926 95.126)
-		(end 188 96.2)
+		(start 178.676943 95.999)
+		(end 179.314 95.361943)
 		(width 0.2)
 		(layer "F.Cu")
@@
 	)
 	(segment
-		(start 176.5 96.348)
-		(end 176.749 96.099)
+		(start 176.4 96.300001)
+		(end 176.701001 95.999)
 		(width 0.2)
 		(layer "F.Cu")
@@
 	)
 	(segment
-		(start 195.2 95.275)
-		(end 195.81 95.885)
+		(start 179.314 95.361943)
+		(end 179.314 94.791585)
 		(width 0.2)
 		(layer "F.Cu")
@@
 	)
 	(segment
-		(start 186.0835 94.2835)
-		(end 186.926 95.126)
+		(start 196.342852 96.450752)
+		(end 204.874 96.450752)
 		(width 0.2)
 		(layer "F.Cu")
@@
 	)
 	(segment
-		(start 181.573951 94.2835)
-		(end 186.0835 94.2835)
+		(start 205.650752 95.674)
+		(end 206.749248 95.674)
 		(width 0.2)
 		(layer "F.Cu")
@@
 	)
 	(segment
-		(start 192.434314 96.2)
-		(end 193.359314 95.275)
+		(start 176.701001 95.999)
+		(end 178.676943 95.999)
 		(width 0.2)
 		(layer "F.Cu")
@@
 	)
 	(segment
-		(start 179.758451 96.099)
-		(end 181.573951 94.2835)
+		(start 192.7469 95.886)
+		(end 189.0909 95.886)
 		(width 0.2)
 		(layer "F.Cu")
@@
 	)
 	(segment
-		(start 207.875 95.675)
-		(end 209.2 97)
+		(start 189.0909 95.886)
+		(end 186.8339 93.629)
 		(width 0.2)
 		(layer "F.Cu")
@@
 	)
 	(segment
-		(start 209.2 97)
-		(end 218.2 97)
+		(start 195.1661 95.274)
+		(end 196.342852 96.450752)
+		(width 0.2)
+		(layer "F.Cu")
+		(net 15)
+	)
+	(segment
+		(start 179.314 94.791585)
+		(end 180.476585 93.629)
 		(width 0.2)
 		(layer "F.Cu")
@@
 	)
 	(segment
-		(start 195.81 95.885)
-		(end 205.315 95.885)
+		(start 193.3589 95.274)
+		(end 192.7469 95.886)
 		(width 0.2)
 		(layer "F.Cu")
@@
 	)
 	(segment
-		(start 176.5 97)
-		(end 176.5 96.348)
+		(start 176.4 96.9)
+		(end 176.4 96.300001)
 		(width 0.2)
 		(layer "F.Cu")
@@
 	)
 	(segment
-		(start 193.359314 95.275)
-		(end 195.2 95.275)
+		(start 204.874 96.450752)
+		(end 205.650752 95.674)
 		(width 0.2)
 		(layer "F.Cu")
@@
 	)
 	(segment
-		(start 205.315 95.885)
-		(end 205.525 95.675)
+		(start 180.476585 93.629)
+		(end 186.8339 93.629)
 		(width 0.2)
 		(layer "F.Cu")
@@
 		(polygon
 			(pts
-				(xy 224 89) (xy 224 114.5) (xy 124.5 114.5) (xy 124.5 89)
+				(xy 224.5 89) (xy 224.5 114.5) (xy 124.5 114.5) (xy 124.5 89)
 			)
 		)
