File: Muon-Boards/Muon-8ch-48.8mm/Muon-8ch-48.8mm.kicad_pcb (KiCad board)
At the start: 4 copper layers, 420.4 x 48.8 mm, 21 parts

Commit message: Added CAEN-8ch-80mm
Parts:
- REF**: moved to F.Cu
- moved REF** 1.86 mm to (-3.00, 93.0)
Connections:
- REF** pad 1: TEMP_OUT -> GND
- REF** pad 2: HV -> TEMP_OUT
- REF** pad 3: GND -> HV
Routing:
- net GND: track 78.7 -> 74.1 mm
- net TEMP_OUT: track 12.3 -> 8.33 mm
- net HV: track 9.69 -> 10.9 mm
Other:
- board text added: "1.3 mm SiPMs S14160-1315PS 48.8 x 48.8 mm2 scint cells Version 4"
- board text removed: "1.3 mm SiPMs S14160-1315PS 48.8 x 48.8 mm2 scint cells Version 3"

Commit message: Added Edge-Card-CAEN
Other:
- copper layers 4 -> 2
Changed lines of the file:
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@@
 	(layers
 		(0 "F.Cu" signal)
-		(4 "In1.Cu" signal)
-		(6 "In2.Cu" signal)
 		(2 "B.Cu" signal)
 		(9 "F.Adhes" user "F.Adhesive")
@@
 			)
 			(layer "dielectric 1"
-				(type "prepreg")
-				(thickness 0.1)
+				(type "core")
+				(thickness 1.51)
 				(material "FR4")
 				(epsilon_r 4.5)
-				(loss_tangent 0.02)
-			)
-			(layer "In1.Cu"
-				(type "copper")
-				(thickness 0.035)
-			)
-			(layer "dielectric 2"
-				(type "core")
-				(thickness 1.24)
-				(material "FR4")
-				(epsilon_r 4.5)
-				(loss_tangent 0.02)
-			)
-			(layer "In2.Cu"
-				(type "copper")
-				(thickness 0.035)
-			)
-			(layer "dielectric 3"
-				(type "prepreg")
-				(thickness 0.1)
-				(material "FR4")
-				(epsilon_r 4.5)
