File: ZDC-Boards/ZDC_Even_Middle_PCB/ZDC_Even_Middle_PCB.kicad_pcb (KiCad board)
At the start: 2 copper layers, 195.2 x 643 mm, 102 parts

Commit message: Updated small connector on ZDC PCBs
Parts:
- added G***: LOGO, LOGO, F.Cu at (45.0, -599.0)
Other:
- outline, holes or cut-outs redrawn
