File: ZDC-Boards/ZDC_Even_Right_PCB/ZDC_Even_Right_PCB.kicad_pcb (KiCad board)
At the start: 2 copper layers, 178.2 x 643 mm, 78 parts

Commit message: Updated small connector on ZDC PCBs
Parts:
- removed the REF** at (131.2, -635.6)
- added G***: LOGO, LOGO, F.Cu at (45.0, -599.0)
- added REF**: PinHeader_2x15_P1.27mm_Horizontal, Connector_PinHeader_1.27mm:PinHeader_2x15_P1.27mm_Horizontal, F.Cu at (131.2, -635.6)
- moved REF**20 2.50 mm to (151.0, -636.0)
Routing:
- net A5: track 681.9 -> 4092.1 mm
- net A11: track 1295.7 -> 647.9 mm
- net A10: track 1193.4 -> 596.7 mm
- net A9: track 1091.1 -> 545.6 mm
- net A8: track 988.8 -> 494.4 mm
- net A7: track 886.5 -> 443.3 mm
- net A6: track 784.2 -> 392.1 mm
- net A4: track 580.5 -> 290.2 mm
Other:
- outline, holes or cut-outs redrawn
