File: ZDC-Boards/ZDC_Even_Right_PCB/ZDC_Even_Right_PCB.kicad_pcb (KiCad board)
At the start: 2 copper layers, 178.2 x 643 mm, 79 parts

Commit message: Updated ZDC connectors to pad connections, v2.0
Parts:
- removed REF**: PinHeader_2x25_P1.27mm_Horizontal, Connector_PinHeader_1.27mm:PinHeader_2x25_P1.27mm_Horizontal
- removed REF**: PinHeader_2x15_P1.27mm_Horizontal, Connector_PinHeader_1.27mm:PinHeader_2x15_P1.27mm_Horizontal
- added J1: TE_5-104895-5_AMPMODU_50-50_2x25_P1.27mm_Horizontal_SMD, TE_AMPMODU:TE_5-104895-5_AMPMODU_50-50_2x25_P1.27mm_Horizontal_SMD, F.Cu at (48.8, -634.4)
- added J2: TE_5-104895-3_AMPMODU_50-50_2x15_P1.27mm_Horizontal_SMD, TE_AMPMODU:TE_5-104895-3_AMPMODU_50-50_2x15_P1.27mm_Horizontal_SMD, F.Cu at (140.1, -634.4)
- #MK1, #MK2: renamed from REF**20; footprint SiPM:S14160-1315PS_dimple_silkscreen_with_capacitor -> SiPM:S14160-1315PS_silkscreen_marker
- C0, C1, C10, C11, C12, C13, C14, C15, C16, C17, C18, C19, C2, C20, C21, C22, C23, C24, C25, C26, C27, C28, C29, C3, C30, C31, C32, C33, C34, C35, C4, C5, C6, C7, C8, C9: renamed from 10 nF
- J3: renamed from REF**; footprint Connector_Coaxial:BNC_TEConnectivity_1478035_Horizontal -> ZDC:BNC_TEConnectivity_1478035_Horizontal_EdgePads
- renumbered REF**20 to D0, REF**20 to D1, REF**20 to D10, REF**20 to D11, REF**20 to D12, REF**20 to D13, REF**20 to D14, REF**20 to D15, REF**20 to D16, REF**20 to D17, REF**20 to D18, REF**20 to D19, REF**20 to D2, REF**20 to D20, REF**20 to D21, REF**20 to D22, REF**20 to D23, REF**20 to D24, REF**20 to D25, REF**20 to D26, REF**20 to D27, REF**20 to D28, REF**20 to D29, REF**20 to D3, REF**20 to D30, REF**20 to D31, REF**20 to D32, REF**20 to D33, REF**20 to D34, REF**20 to D35, REF**20 to D4, REF**20 to D5, REF**20 to D6, REF**20 to D7, REF**20 to D8, REF**20 to D9, REF** to J4
Connections:
- C24 pad 1: K0 -> K24
- C25 pad 1: K1 -> K25
- C26 pad 1: K2 -> K26
- C27 pad 1: K3 -> K27
- C28 pad 1: K4 -> K28
- C29 pad 1: K5 -> K29
- C30 pad 1: K6 -> K30
- C31 pad 1: K7 -> K31
- C32 pad 1: K8 -> K32
- C33 pad 1: K9 -> K33
- C34 pad 1: K10 -> K34
- C35 pad 1: K11 -> K35
- D0 pad : LK -> LK1
- D0 pad 7: (no net) -> K0
- D0 pad 8: (no net) -> A0
- D0 pad 9: LA -> LA1
- D1 pad : LK -> LK1
- D1 pad 7: (no net) -> K1
- D1 pad 8: (no net) -> A1
- D1 pad 9: LA -> LA1
- D10 pad : LK -> LK1
- D10 pad 7: (no net) -> K10
- D10 pad 8: (no net) -> A10
- D10 pad 9: LA -> LA1
- D11 pad : LK -> LK1
- D11 pad 7: (no net) -> K11
- D11 pad 8: (no net) -> A11
- D11 pad 9: LA -> LA1
- D12 pad : LK -> LK1
- D12 pad 9: LA -> LA1
- D13 pad : LK -> LK1
- D13 pad 7: (no net) -> K13
- D13 pad 8: (no net) -> A13
- D13 pad 9: LA -> LA1
- D14 pad : LK -> LK1
- D14 pad 7: (no net) -> K14
- D14 pad 8: (no net) -> A14
- D14 pad 9: LA -> LA1
- D15 pad : LK -> LK1
- D15 pad 7: (no net) -> K15
- D15 pad 8: (no net) -> A15
- D15 pad 9: LA -> LA1
- D16 pad : LK -> LK1
- D16 pad 7: (no net) -> K16
- D16 pad 8: (no net) -> A16
- D16 pad 9: LA -> LA1
- D17 pad : LK -> LK1
- D17 pad 7: (no net) -> K17
- D17 pad 9: LA -> LA1
- D18 pad : LK -> LK1
- D18 pad 7: (no net) -> K18
- D18 pad 8: (no net) -> A18
- D18 pad 9: LA -> LA1
- D19 pad : LK -> LK1
- D19 pad 7: (no net) -> K19
- D19 pad 8: (no net) -> A19
- D19 pad 9: LA -> LA1
- D2 pad : LK -> LK1
- D2 pad 7: (no net) -> K2
- D2 pad 8: (no net) -> A2
- D2 pad 9: LA -> LA1
- D20 pad : LK -> LK1
- D20 pad 7: (no net) -> K20
- D20 pad 8: (no net) -> A20
- D20 pad 9: LA -> LA1
- D21 pad : LK -> LK1
- D21 pad 7: (no net) -> K21
- D21 pad 8: (no net) -> A21
- D21 pad 9: LA -> LA1
- D22 pad : LK -> LK1
- D22 pad 7: (no net) -> K22
- D22 pad 8: (no net) -> A22
- D22 pad 9: LA -> LA1
- D23 pad : LK -> LK1
- D23 pad 7: (no net) -> K23
- D23 pad 8: (no net) -> A23
- D23 pad 9: LA -> LA1
- D24 pad : LK -> LK2
- D24 pad 7: (no net) -> K24
- D24 pad 8: (no net) -> A24
- D24 pad 9: LA -> LA2
- D25 pad : LK -> LK2
- D25 pad 7: (no net) -> K25
- D25 pad 8: (no net) -> A25
- D25 pad 9: LA -> LA2
- D26 pad : LK -> LK2
- D26 pad 7: (no net) -> K26
- D26 pad 8: (no net) -> A26
- D26 pad 9: LA -> LA2
- D27 pad : LK -> LK2
- D27 pad 7: (no net) -> K27
- D27 pad 8: (no net) -> A27
- D27 pad 9: LA -> LA2
- D28 pad : LK -> LK2
- D28 pad 7: (no net) -> K28
- D28 pad 8: (no net) -> A28
- D28 pad 9: LA -> LA2
- D29 pad : LK -> LK2
- D29 pad 7: (no net) -> K29
- D29 pad 8: A5 -> A29
- D29 pad 9: LA -> LA2
- D3 pad : LK -> LK1
- D3 pad 7: (no net) -> K3
- D3 pad 8: (no net) -> A3
- D3 pad 9: LA -> LA1
- D30 pad : LK -> LK2
- D30 pad 7: (no net) -> K30
- D30 pad 8: (no net) -> A30
- D30 pad 9: LA -> LA2
- D31 pad : LK -> LK2
- D31 pad 7: (no net) -> K31
- D31 pad 8: (no net) -> A31
- D31 pad 9: LA -> LA2
- D32 pad : LK -> LK2
- D32 pad 7: (no net) -> K32
- D32 pad 8: (no net) -> A32
- D32 pad 9: LA -> LA2
- D33 pad : LK -> LK2
- D33 pad 7: (no net) -> K33
- D33 pad 8: (no net) -> A33
- D33 pad 9: LA -> LA2
- D34 pad : LK -> LK2
- D34 pad 7: (no net) -> K34
- D34 pad 8: (no net) -> A34
- D34 pad 9: LA -> LA2
- D35 pad : LK -> LK2
- D35 pad 7: (no net) -> K35
- D35 pad 8: (no net) -> A35
- D35 pad 9: LA -> LA2
- D4 pad : LK -> LK1
- D4 pad 7: (no net) -> K4
- D4 pad 8: (no net) -> A4
- D4 pad 9: LA -> LA1
- D5 pad : LK -> LK1
- D5 pad 7: (no net) -> K5
- D5 pad 9: LA -> LA1
- D6 pad : LK -> LK1
- D6 pad 7: (no net) -> K6
- D6 pad 8: (no net) -> A6
- D6 pad 9: LA -> LA1
- D7 pad : LK -> LK1
- D7 pad 7: (no net) -> K7
- D7 pad 8: (no net) -> A7
- D7 pad 9: LA -> LA1
- D8 pad : LK -> LK1
- D8 pad 7: (no net) -> K8
- D8 pad 8: (no net) -> A8
- D8 pad 9: LA -> LA1
- D9 pad : LK -> LK1
- D9 pad 7: (no net) -> K9
- D9 pad 8: (no net) -> A9
- D9 pad 9: LA -> LA1
- J3 pad 1: LA -> LA1
- J3 pad 2: LK -> LK1
- J4 pad 1: LA -> LA2
- J4 pad 2: LK -> LK2
Routing:
- net A5: track 4092.1 -> 350.4 mm
- net LK: track 1979.9 -> 0.00 mm, vias 36 -> 0
- net LA: track 1896.2 -> 0.00 mm, vias 4 -> 0
- net LK1: track 0.00 -> 1315.8 mm, vias 0 -> 24
- net LA1: track 0.00 -> 1265.0 mm, vias 0 -> 2
- net LK2: track 0.00 -> 660.0 mm, vias 0 -> 12
- net A35: track 0.00 -> 657.6 mm
- net LA2: track 0.00 -> 625.4 mm
- net K11: track 1248.1 -> 622.9 mm, vias 4 -> 2
- net K35: track 0.00 -> 622.9 mm, vias 0 -> 2
- net A34: track 0.00 -> 606.3 mm
- net K10: track 1149.0 -> 573.3 mm, vias 4 -> 2
- net K34: track 0.00 -> 573.3 mm, vias 0 -> 2
- net A33: track 0.00 -> 554.9 mm
- net K33: track 0.00 -> 525.2 mm, vias 0 -> 2
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- added copper zone on B.Cu, net (none)
- added copper zone on F.Cu, net (none)
Other:
- board text added: "TE 5-104895-3 (AMPMODU 50/50 R/A SMT)"
- board text added: "TE 5-104895-5 (AMPMODU 50/50 R/A SMT)"
- board text added: "ZDC Even Right PCB v2.0 Designed by Sean Preins"
- board text removed: "ZDC Even Right PCB v1.0 Designed by Sean Preins"

Commit message: Updated ZDC boards to use new pin connectors that attach to crimped cables
Parts:
- J1: value TE_5-104895-5_AMPMODU_50-50_2x25_P1.27mm_Horizontal_SMD -> Samtec_TFM-125-01-x-D-RE1-WT_2x25_P1.27mm_Horizontal; footprint TE_AMPMODU:TE_5-104895-5_AMPMODU_50-50_2x25_P1.27mm_Horizontal_SMD -> Samtec_TFM:Samtec_TFM-125-01-x-D-RE1-WT_2x25_P1.27mm_Horizontal
- J2: value TE_5-104895-3_AMPMODU_50-50_2x15_P1.27mm_Horizontal_SMD -> Samtec_TFM-115-01-x-D-RE1-WT_2x15_P1.27mm_Horizontal; footprint TE_AMPMODU:TE_5-104895-3_AMPMODU_50-50_2x15_P1.27mm_Horizontal_SMD -> Samtec_TFM:Samtec_TFM-115-01-x-D-RE1-WT_2x15_P1.27mm_Horizontal
- moved #MK1 3.42 mm to (69.4, -636.0)
- moved #MK2 3.32 mm to (154.3, -636.0)
- moved J1 1.34 mm to (48.8, -635.7), turned to 0 degrees
- moved J2 1.34 mm to (140.1, -635.7), turned to 0 degrees
Connections:
- J1 pad 10: A3 -> K20
- J1 pad 11: K4 -> A19
- J1 pad 12: A4 -> K19
- J1 pad 13: K5 -> A18
- J1 pad 14: A5 -> K18
- J1 pad 15: K6 -> A17
- J1 pad 16: A6 -> K17
- J1 pad 17: K7 -> A16
- J1 pad 18: A7 -> K16
- J1 pad 19: K8 -> A15
- J1 pad 20: A8 -> K15
- J1 pad 21: K9 -> A14
- J1 pad 22: A9 -> K14
- J1 pad 23: K10 -> A13
- J1 pad 24: A10 -> K13
- J1 pad 25: K11 -> A12
- J1 pad 26: A11 -> K12
- J1 pad 27: K12 -> A11
- J1 pad 28: A12 -> K11
- J1 pad 29: K13 -> A10
- J1 pad 3: K0 -> A23
- J1 pad 30: A13 -> K10
- J1 pad 31: K14 -> A9
- J1 pad 32: A14 -> K9
- J1 pad 33: K15 -> A8
- J1 pad 34: A15 -> K8
- J1 pad 35: K16 -> A7
- J1 pad 36: A16 -> K7
- J1 pad 37: K17 -> A6
- J1 pad 38: A17 -> K6
- J1 pad 39: K18 -> A5
- J1 pad 4: A0 -> K23
- J1 pad 40: A18 -> K5
- J1 pad 41: K19 -> A4
- J1 pad 42: A19 -> K4
- J1 pad 43: K20 -> A3
- J1 pad 44: A20 -> K3
- J1 pad 45: K21 -> A2
- J1 pad 46: A21 -> K2
- J1 pad 47: K22 -> A1
- J1 pad 48: A22 -> K1
- J1 pad 49: K23 -> A0
- J1 pad 5: K1 -> A22
- J1 pad 50: A23 -> K0
- J1 pad 6: A1 -> K22
- J1 pad 7: K2 -> A21
- J1 pad 8: A2 -> K21
- J1 pad 9: K3 -> A20
- J2 pad 10: A27 -> K34
- J2 pad 11: K28 -> A33
- J2 pad 12: A28 -> K33
- J2 pad 13: K29 -> A32
- J2 pad 14: A29 -> K32
- J2 pad 15: K30 -> A31
- J2 pad 16: A30 -> K31
- J2 pad 17: K31 -> A30
- J2 pad 18: A31 -> K30
- J2 pad 19: K32 -> A29
- J2 pad 20: A32 -> K29
- J2 pad 21: K33 -> A28
- J2 pad 22: A33 -> K28
- J2 pad 23: K34 -> A27
- J2 pad 24: A34 -> K27
- J2 pad 25: K35 -> A26
- J2 pad 26: A35 -> K26
- J2 pad 27: (no net) -> A25
- J2 pad 28: (no net) -> K25
- J2 pad 29: (no net) -> A24
- J2 pad 3: K24 -> (no net)
- J2 pad 30: (no net) -> K24
- J2 pad 4: A24 -> (no net)
- J2 pad 5: K25 -> (no net)
- J2 pad 6: A25 -> (no net)
- J2 pad 7: K26 -> A35
- J2 pad 8: A26 -> K35
- J2 pad 9: K27 -> A34
- J2 pad MP: (no net) -> GND
Routing:
- net A6: track 402.0 -> 392.3 mm, vias 0 -> 1
- net A30: track 402.0 -> 392.3 mm, vias 0 -> 1
- net A7: track 452.1 -> 444.3 mm, vias 0 -> 1
- net A31: track 452.1 -> 444.3 mm, vias 0 -> 1
- net A8: track 503.5 -> 496.3 mm, vias 0 -> 1
- net A32: track 503.5 -> 496.3 mm, vias 0 -> 1
- net A2: track 195.7 -> 189.7 mm
- net A26: track 195.7 -> 189.7 mm
- net A9: track 554.9 -> 549.1 mm, vias 0 -> 1
- net A33: track 554.9 -> 549.1 mm, vias 0 -> 1
- net A1: track 144.1 -> 138.3 mm
- net A25: track 144.1 -> 138.3 mm
- net A0: track 93.1 -> 87.6 mm
- net A24: track 93.1 -> 87.6 mm
- net A10: track 606.3 -> 601.1 mm, vias 0 -> 1
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Other:
- board text added: "Samtec TFM-115-01-L-D-RE1-WT"
- board text added: "Samtec TFM-125-01-L-D-RE1-WT"
- board text removed: "TE 5-104895-3 (AMPMODU 50/50 R/A SMT)"
- board text removed: "TE 5-104895-5 (AMPMODU 50/50 R/A SMT)"
