File: ZDC-Boards/ZDC_Odd_Right_PCB/ZDC_Odd_Right_PCB.kicad_pcb (KiCad board)
At the start: 2 copper layers, 202.6 x 643 mm, 94 parts

Commit message: Updated small connector on ZDC PCBs
Parts:
- added G***: LOGO, LOGO, F.Cu at (45.0, -599.0)
Other:
- outline, holes or cut-outs redrawn
